File: HARDWARE/NeuroBytes_Vestibular_System.sch (KiCad schematic (older format))
At the start: 28 parts, among them P1 JST GH 4-POS, P5 JST GH 4-POS, P6 JST GH 4-POS, P7 JST GH 4-POS, P8 JST GH 7-POS, Q1 NPN_dual, Q2 NPN_dual, SW1 SW_PUSH_TL3330AF130QG, U1 STM32L011Gx, U2 LD3985G33R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

Commit message: Updated graphics to improve 3D orthoganol canal effect.
Parts:
- removed Q1: NPN_dual, KiCad_Footprints:ZF_SMD_SOT-363, symbol NPN_dual
- removed RN1: 1k_x4, KiCad_Footprints:ZF_RN_4iso_CTS-0804, symbol R_Pack04
- removed RN3: 100_x4, KiCad_Footprints:ZF_RN_4iso_CTS-0804, symbol R_Pack04
- added D5: LED, KiCad_Footprints:ZF_SMD_NonPol_0402, symbol LED
- added P2: JST GH 4-POS, KiCad_Footprints:ZF_CONN_JST_GH, symbol CONN_01X04
- added R1, R2, R3, R5, R6, R7, R8: R, KiCad_Footprints:ZF_SMD_NonPol_0402, symbol R
- added SW2: Switch_DPDT, KiCad_Footprints:ZF_SW_Slide_DPDT_SMD, symbol Switch_DPDT
Connections:
- net LED_0 is gone; now on net LED_X0: U1.7 (PA1_5V/TIM2_CH2)
- net LED_1 is gone; now on net LED_X1: U1.6 (PA0_3V3/TIM2_CH1)
- net +5V: now also P2.2 (P2); no longer D1.2 (A), D2.2 (A), D3.2 (A), D4.2 (A)
- net A2EX: now also U1.15 (PB1_5V/MOSI/TIM2_CH4); no longer U1.25 (PB4_5V)
- net A4EX: now also U1.11 (PA5_3V3/TIM2_CH1); no longer U1.9 (PA3_5V/TIM2_CH4/TIM21_CH2)
- net A4IN: now also U1.10 (PA4_3V3/NSS); no longer U1.8 (PA2_3V3/TIM2_CH3/TIM21_CH1)
- net GND: now also P2.1 (P1), SW2.2
- net INT: now also U1.25 (PB4_5V); no longer U1.11 (PA5_3V3/TIM2_CH1)
- net MOSI: now also SW2.1
- net at Q2.2 (BASE2): now also R2.1
- net at Q2.3: now also R7.1, R8.1
- net at Q2.5 (BASE1): now also R1.1
- net at Q2.6: now also R3.1, R5.1, R6.1
- net LED_Y0: now reaches U1.14 (PB0_5V/TIM2_CH2/3)
- net LED_Y0: now also R1.2
- net LED_X1: now reaches D4.1 (K)
- net LED_X1: now also D3.1 (K)
- net LED_X0: now reaches D2.1 (K)
- net LED_X0: now also D1.1 (K)
- net LED_2 renamed LED_X2
- net LED_X2: now also D5.1 (K)
- net LED_3 renamed LED_Y1
- net LED_Y1: now also R2.2
- net nRESET: no longer names the net of RN2.7 (R2.2), U3.11 (nRESET)
- net nRESET: no longer U1.10 (PA4_3V3/NSS)
- new net: D4.2 (A), R8.2
- new net: D3.2 (A), R5.2
- new net: D2.2 (A), R7.2
- new net: D1.2 (A), R3.2
- new net: D5.2 (A), R6.2
- new net A5EX: P2.4 (P4), U1.9 (PA3_5V/TIM2_CH4/TIM21_CH2)
- new net A5IN: P2.3 (P3), U1.8 (PA2_3V3/TIM2_CH3/TIM21_CH1)
Other:
- moved on the sheet: C1, C4, D1, D2, D3, D4, P8, Q2, U2

Commit message: first PCB routing revision.
Parts:
- removed RN2: 10k_x4, KiCad_Footprints:ZF_RN_4iso_CTS-0804, symbol R_Pack04
- removed SW2: Switch_DPDT, KiCad_Footprints:ZF_SW_Slide_DPDT_SMD, symbol Switch_DPDT
- added D10, D11, D12, D6, D7, D8, D9: LED, KiCad_Footprints:ZF_SMD_NonPol_0402, symbol LED
- added Q1: NPN_dual, KiCad_Footprints:ZF_SMD_SOT-363, symbol NPN_dual
- added RN1, RN3: 100 x4, KiCad_Footprints:ZF_RN_4iso_CTS-0804, symbol R_Pack04
- added RN4: 150 x4, KiCad_Footprints:ZF_RN_4iso_CTS-0804, symbol R_Pack04
- R5, R6, R7, R8: value R -> 10k
Connections:
- net MOSI is gone; now on net IDENTIFY: P8.6 (P6), U1.26 (PB5_5V/MOSI/TIM21_CH1)
- net +3V3: now also R5.2, R6.2, R7.2, R8.2
- net A1EX: now also U1.25 (PB4_5V); no longer U1.18 (PA8_5V/TIM2_CH1)
- net A1IN: now also U1.24 (PB3_5V/TIM2_CH2); no longer U1.3 (PC15_3V3)
- net A2EX: now also U1.12 (PA6_5V); no longer U1.15 (PB1_5V/MOSI/TIM2_CH4)
- net A2IN: now also U1.11 (PA5_3V3/TIM2_CH1); no longer U1.12 (PA6_5V)
- net A3EX: now also U1.8 (PA2_3V3/TIM2_CH3/TIM21_CH1); no longer U1.2 (PC14_5V)
- net A3IN: now also U1.6 (PA0_3V3/TIM2_CH1); no longer U1.13 (PA7_5V/MOSI)
- net A4EX: now also U1.15 (PB1_5V/MOSI/TIM2_CH4); no longer U1.11 (PA5_3V3/TIM2_CH1)
- net A4IN: now also U1.13 (PA7_5V/MOSI); no longer U1.10 (PA4_3V3/NSS)
- net A5EX: now also U1.3 (PC15_3V3); no longer U1.9 (PA3_5V/TIM2_CH4/TIM21_CH2)
- net A5IN: now also U1.2 (PC14_5V); no longer U1.8 (PA2_3V3/TIM2_CH3/TIM21_CH1)
- net GND: now also Q1.1; no longer U3.10 (PIN10)
- net IDENTIFY: no longer U1.24 (PB3_5V/TIM2_CH2)
- net LED_X0: now also U1.18 (PA8_5V/TIM2_CH1), D11.1 (K), D8.1 (K); no longer D2.1 (K), U1.7 (PA1_5V/TIM2_CH2)
- net LED_X1: now also U1.28 (PB7_5V/TIM2_CH4), D12.1 (K), D7.1 (K); no longer D4.1 (K), U1.6 (PA0_3V3/TIM2_CH1)
- net LED_X2: now also D4.1 (K), U1.7 (PA1_5V/TIM2_CH2), D10.1 (K); no longer U1.28 (PB7_5V/TIM2_CH4)
- net LED_Y0: now also R3.2; no longer R1.2
- net LED_Y1: now also R1.2, U1.9 (PA3_5V/TIM2_CH4/TIM21_CH2); no longer R2.2, U1.27 (PB6_5V/TIM2_CH3)
- net SCL: now also R8.1
- net SDA: now also R7.1
- net at D4.2 (A): now also RN3.7 (R2.2); no longer R8.2
- net at D3.2 (A): now also RN1.7 (R2.2); no longer R5.2
- net at D2.2 (A): now also RN3.8 (R1.2); no longer R7.2
- net at D1.2 (A): now also RN1.8 (R1.2); no longer R3.2
- net at U3.11 (nRESET): now also R6.1
- net at U3.4 (nBOOT_LOAD): now also R5.1
- net at D5.2 (A): now also RN1.6 (R3.2); no longer R6.2
- net INT: no longer names the net of U3.14 (INT)
- net INT: no longer U1.25 (PB4_5V)
- new net: Q2.3, RN3.1 (R1.1), RN3.2 (R2.1), RN3.3 (R3.1), RN3.4 (R4.1)
- new net: Q2.6, RN1.1 (R1.1), RN1.2 (R2.1), RN1.3 (R3.1), RN1.4 (R4.1)
- new net: D6.2 (A), RN1.5 (R4.2)
- new net: D8.2 (A), RN3.5 (R4.2)
- new net: D7.2 (A), RN3.6 (R3.2)
- new net: Q1.2 (BASE2), R3.1
- new net: Q1.6, RN4.1 (R1.1), RN4.2 (R2.1), RN4.3 (R3.1), RN4.4 (R4.1)
- new net: D10.2 (A), RN4.7 (R2.2)
- new net: D9.2 (A), RN4.8 (R1.2)
- new net: D11.2 (A), RN4.5 (R4.2)
- new net: D12.2 (A), RN4.6 (R3.2)
- new net LED_X3: D2.1 (K), D6.1 (K), D9.1 (K), U1.27 (PB6_5V/TIM2_CH3)
- new net LED_Y2: R2.2, U1.10 (PA4_3V3/NSS)
Other:
- moved on the sheet: D2, D3, D4, D5, P1, P2, P5, P6, P7, SW1

Commit message: reversed LEDs
Connections:
- net LED_X0: now also D1.2 (A), D11.2 (A), D8.2 (A); no longer D1.1 (K), D11.1 (K), D8.1 (K)
- net LED_X1: now also D12.2 (A), D3.2 (A), D7.2 (A); no longer D12.1 (K), D3.1 (K), D7.1 (K)
- net LED_X2: now also D10.2 (A), D4.2 (A), D5.2 (A); no longer D10.1 (K), D4.1 (K), D5.1 (K)
- net LED_X3: now also D2.2 (A), D6.2 (A), D9.2 (A); no longer D2.1 (K), D6.1 (K), D9.1 (K)
- net at RN3.7 (R2.2): now also D4.1 (K); no longer D4.2 (A)
- net at RN1.7 (R2.2): now also D3.1 (K); no longer D3.2 (A)
- net at RN3.8 (R1.2): now also D2.1 (K); no longer D2.2 (A)
- net at RN1.8 (R1.2): now also D1.1 (K); no longer D1.2 (A)
- net at RN1.6 (R3.2): now also D5.1 (K); no longer D5.2 (A)
- net at RN1.5 (R4.2): now also D6.1 (K); no longer D6.2 (A)
- net at RN3.5 (R4.2): now also D8.1 (K); no longer D8.2 (A)
- net at RN3.6 (R3.2): now also D7.1 (K); no longer D7.2 (A)
- net at RN4.7 (R2.2): now also D10.1 (K); no longer D10.2 (A)
- net at RN4.8 (R1.2): now also D9.1 (K); no longer D9.2 (A)
- net at RN4.5 (R4.2): now also D11.1 (K); no longer D11.2 (A)
- net at RN4.6 (R3.2): now also D12.1 (K); no longer D12.2 (A)
Other:
- moved on the sheet: D1, D10, D11, D12, D2, D3, D4, D5, D6, D7, D8, D9
Changed lines of the file:
@@
 F 5 "Yes" H 10650 4500 60  0001 C CNN "RoHS"
 	1    10650 4500
-	0    -1   -1   0
+	0    1    1    0
 $EndComp
 $Comp
@@
 P 9650 3900
 F 0 "D3" H 9650 4000 50  0000 C CNN
-F 1 "LED" H 9650 3800 50  0000 C CNN
+F 1 "LED" V 9650 3800 50  0000 C CNN
 F 2 "KiCad_Footprints:ZF_SMD_NonPol_0402" H 9650 3900 50  0001 C CNN
 F 3 "" H 9650 3900 50  0000 C CNN
@@
 F 5 "Yes" H 9650 3900 60  0001 C CNN "RoHS"
 	1    9650 3900
-	0    -1   -1   0
+	0    1    1    0
 $EndComp
 $Comp
@@
 F 5 "Yes" H 10750 5100 60  0001 C CNN "RoHS"
 	1    10750 5100
-	0    -1   -1   0
+	0    1    1    0
 $EndComp
 $Comp
@@
 F 5 "Yes" H 9550 3300 60  0001 C CNN "RoHS"
 	1    9550 3300
-	0    -1   -1   0
+	0    1    1    0
 $EndComp
 $Comp
@@
 F 5 "Yes" H 9750 4500 60  0001 C CNN "RoHS"
 	1    9750 4500
-	0    -1   -1   0
+	0    1    1    0
 $EndComp
 $Comp
@@
 F 5 "Yes" H 9850 5100 60  0001 C CNN "RoHS"
 	1    9850 5100
-	0    -1   -1   0
+	0    1    1    0
 $EndComp
 Wire Wire Line
@@
 F 5 "Yes" H 10550 3900 60  0001 C CNN "RoHS"
 	1    10550 3900
-	0    -1   -1   0
+	0    1    1    0
 $EndComp
 Wire Wire Line
@@
 F 5 "Yes" H 10450 3300 60  0001 C CNN "RoHS"
 	1    10450 3300
-	0    -1   -1   0
+	0    1    1    0
 $EndComp
 Wire Wire Line
@@
 F 5 "Yes" H 11550 4500 60  0001 C CNN "RoHS"
 	1    11550 4500
-	0    -1   -1   0
+	0    1    1    0
 $EndComp
 $Comp
@@
 F 5 "Yes" H 11650 5100 60  0001 C CNN "RoHS"
 	1    11650 5100
-	0    -1   -1   0
+	0    1    1    0
 $EndComp
 Wire Wire Line
@@
 F 5 "Yes" H 11350 3300 60  0001 C CNN "RoHS"
 	1    11350 3300
-	0    -1   -1   0
+	0    1    1    0
 $EndComp
 Wire Wire Line
@@
 F 5 "Yes" H 11450 3900 60  0001 C CNN "RoHS"
 	1    11450 3900
-	0    -1   -1   0
-$EndComp
-Wire Wire Line
+	0    1    1    0
+$EndComp
+Wire Wire Line
